Commit message: gazebo sim

File: dev_ws/src/my_bot/description/my_bot.urdf.xacro (robot description, xacro)
@@ -2,3 +2,4 @@
 <robot xmlns:xacro="http://www.ros.org/wiki/xacro" name="my_bot"> <!--(name doesn't need to match file name)-->
     <xacro:include filename="robot_core.xacro"/>
+    <xacro:include filename="gazebo_control.xacro"/>
 </robot>

File: dev_ws/src/my_bot/description/robot_core.xacro (robot description, xacro)
@@ -27,5 +27,5 @@
                 <box size="${body_length} ${body_width} ${body_height}"/>
             </geometry>
-            <material name="red"/>
+            <material name="white"/>
         </visual>
         <collision>
@@ -39,4 +39,7 @@
         </xacro:inertial_box>
     </link>
+    <gazebo reference="body_link">
+        <material>Gazebo/White</material>
+    </gazebo>
     <!-- Drive wheels -->
     <!-- Left Wheel -->
@@ -63,4 +66,7 @@
         </xacro:inertial_cylinder>
     </link>
+    <gazebo reference="left_wheel_link">
+        <material>Gazebo/Blue</material>
+    </gazebo>
     <!-- Right Wheel -->
     <joint name="right_wheel_joint" type="continuous">
@@ -68,5 +74,5 @@
         <child link="right_wheel_link"/>
         <origin xyz="0 -${body_width/2+wheel_width/2} ${wheel_zoffset}" rpy="${pi/2} 0 0"/>
-        <axis xyz="0 0 1"/>
+        <axis xyz="0 0 -1"/>
     </joint>
     <link name="right_wheel_link">
@@ -86,4 +92,7 @@
         </xacro:inertial_cylinder>
     </link>
+    <gazebo reference="right_wheel_link">
+        <material>Gazebo/Blue</material>
+    </gazebo>
     <!-- Caster Wheel -->
     <joint name="caster_joint" type="fixed">
@@ -108,3 +117,8 @@
         </xacro:inertial_sphere>
     </link>
+    <gazebo reference="caster_link">
+        <material>Gazebo/Black</material>
+        <mu1 value="0.001"/>
+        <mu2 value="0.001"/>
+    </gazebo>
 </robot>
