Commit message: wip camera + dev-jetson image

File: dev_ws/src/my_bot/description/materials.xacro (robot description, xacro)
@@ -14,3 +14,6 @@
         <color rgba="1 0 0 1"/>
     </material>
+    <material name="green">
+        <color rgba="0 1 0 1"/>
+    </material>
 </robot>

File: dev_ws/src/my_bot/description/my_bot.urdf.xacro (robot description, xacro)
@@ -3,3 +3,4 @@
     <xacro:include filename="robot_core.xacro"/>
     <xacro:include filename="gazebo_control.xacro"/>
+    <xacro:include filename="camera.xacro"/>
 </robot>
